File: driver/driver.kicad_pcb (KiCad board)
At the start: 4 copper layers, 34.8 x 27 mm, 61 parts, among them J101 UJC-HP-3-SMT-TR, J102 fan_header_4pin, J103 TagConnect-2x3, Q102 SiSS63DN, Q104 FDV301N, Q105 SiSS63DN, SW101 A6S-1101-H, U101 STUSB4500QTR, U102 MPM3606, U103 SLG46621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

Commit message: FAN_PWM: guard against high voltage from the fan
Parts:
- added Q101: FDV301N, proj:SOT-23, B.Cu at (94.2, 72.0)
- added R110: 100k, proj:R_0402_1005Metric, B.Cu at (94.6, 74.5)
Connections:
- U103 pad 3: /FAN_PWM -> /FAN_PWM_LV
Routing:
- net /FAN_PWM_LV: track 0.00 -> 10.5 mm, vias 0 -> 2
- net /FAN_PWM: track 12.8 -> 5.29 mm, vias 1 -> 0
- net GND: track 44.0 -> 47.6 mm, vias 35 -> 38
- net /FAN_V_{snk}: track 13.9 -> 15.7 mm
